File: raspi-shield.sch (EAGLE design)
At the start: 1 part, among them K1 PIN20X2

Commit message: added imu/depth/pwm mux
Parts:
- added B1: Pressure Sensor, SparkFun-Boards:SPARKFUN_MS5803-14BA_BREAKOUT
- added J1: (no value), SparkFun-Connectors:CONN_06NO_SILK_FEMALE_PTH
- added J2: (no value), SparkFun-Connectors:CONN_041X04_NO_SILK
- added R1: 10k, SparkFun-Resistors:10KOHM-0603-1/10W-1%
- added U1: PCA9685, SparkFun-IC-Special-Function:PCA9685
Connections:
- new net 3.3V: B1.3.3V, J1.2, U1.VDD
- new net ESTOP: K1.11, R1.2, U1.!OE
- new net PWM0: U1.CH0
- new net PWM1: U1.CH1
- new net PWM10: U1.CH10
- new net PWM11: U1.CH11
- new net PWM12: U1.CH12
- new net PWM13: U1.CH13
- new net PWM14: U1.CH14
- new net PWM15: U1.CH15
- new net PWM2: U1.CH2
- new net PWM3: U1.CH3
- new net PWM4: U1.CH4
- new net PWM5: U1.CH5
- new net PWM6: U1.CH6
- new net PWM7: U1.CH7
- new net PWM8: U1.CH8
- new net PWM9: U1.CH9
- new net SCL: B1.SCL/SCLK, J1.5, K1.5, U1.SCL
- new net SDA: B1.SDA/SDI, J1.4, K1.3, U1.SDA
- net GND: now also B1.GND, J1.3, R1.1, U1.A0, U1.A1, U1.A2, U1.A3, U1.A4, U1.A5, U1.EXTCLK, U1.VSS
Other:
- note added: "Depth"
- note added: "GPIO"
- note added: "IMU"
- note added: "PWM Outputs"
